File: oven-controller.sch (KiCad schematic (older format))
At the start: 20 parts, among them J1 USB, J2 ISP, J3 Thermocouple, J4 Load In, J5 Neut In, U1 ATMEGA16U2, U2 MAX31855KASA, U3 MOC3022S, U4 LTV-354T, Y1 16MHz

Commit message: oven-controller v2
Parts:
- removed C4: 0.1uF, Capacitors_SMD:C_0603_HandSoldering, symbol C
- C1, C2, C3: footprint Capacitors_SMD:C_0603_HandSoldering -> Capacitors_SMD:C_0805_HandSoldering
- J2: footprint Socket_Strips:Socket_Strip_Straight_2x03_Pitch2.54mm -> Pin_Headers:Pin_Header_Straight_2x03_Pitch2.54mm
- R1, R2, R3: footprint Resistors_SMD:R_0402 -> Resistors_SMD:R_0805_HandSoldering
- Y1: footprint Crystals:Crystal_HC52-U_Vertical -> Crystals:Crystal_HC49-U_Vertical
Connections:
- net GND: now also J1.6 (Shield)
- net +3V3: now reaches C3.2, U1.27 (UCAP), U1.32 (AVCC), U1.4 (VCC)
- net +3V3: now also J2.2 (Pin_2), U2.4 (VCC)
- net 3.3V: no longer names the net of U1.18 ((T1/PCINT4)PB4)
- net 3.3V: no longer U2.4 (VCC)
- net VBUS: no longer names the net of J1.1 (VBUS), U1.31 (UVCC)
- net VBUS: no longer J2.2 (Pin_2)
Other:
- note added: "120V * sqrt(2) / 1A\n= 220 ohms\n\n120V * sqrt(2) * 1A\n= 120W * sqrt(2)\n\n120W * sqrt(2) * 5us * 120Hz\n= 0.1 W"
- note removed: "120V * sqrt(2) / 1A\n= 220 ohms\n\n120V * sqrt(2) * 1A\n= 120W * sqrt(2)\n\n120W * sqrt(2) * 4us / (1/120)s\n= 8.15E-2"
- moved on the sheet: R5, U4
